Commit message: added launchpad model

File: multi_jackal_description/urdf/jackal.urdf.xacro (robot description, xacro)
@@ -177,3 +177,31 @@
   <!-- Optional custom accessories. -->
   <xacro:include filename="custom_accessories.urdf.xacro" />
+  <!-- <xacro:include filename="$(find multi_jackal_description)/urdf/_d435.urdf.xacro" />
+  <sensor_d435 parent="base_link" name="rs_d435" topics_ns="$(arg namespace)/rs_d435" >
+    <origin xyz="0.4 0 0.2" rpy="0 0 0" />
+  </sensor_d435>
+  <xacro:include filename="$(find velodyne_description)/urdf/VLP-16.urdf.xacro"/>
+  <VLP-16 parent="base_link" name="velodyne" topic="$(arg namespace)/velodyne_points" hz="10" samples="360" gpu="false" lasers="16" max_range="50">
+    <origin xyz="0 0 0.2" rpy="0 0 0" />
+  </VLP-16> -->
+  <link name="land_pad">
+    <visual>
+      <geometry>
+        <box size="0.56 0.5 0.02"/>
+      </geometry>
+    </visual>
+    <collision>
+      <geometry>
+        <box size="0.56 0.5 0.02"/>
+      </geometry>
+    </collision>
+  </link>
+  <gazebo reference="land_pad">
+    <material>Gazebo/Black</material>
+  </gazebo>
+  <joint name="land_pad_link" type="fixed">
+    <parent link="base_link"/>
+    <child link="land_pad"/>
+    <origin xyz="0 0 0.38" rpy="0 0 0"/>
+  </joint>
 </robot>

Commit message: modifications in order to have velodyne, laser scan, and waypoint navigation.

File: multi_jackal_description/urdf/jackal.urdf.xacro (robot description, xacro)
@@ -180,9 +180,9 @@
   <sensor_d435 parent="base_link" name="rs_d435" topics_ns="$(arg namespace)/rs_d435" >
     <origin xyz="0.4 0 0.2" rpy="0 0 0" />
-  </sensor_d435>
+  </sensor_d435> -->
   <xacro:include filename="$(find velodyne_description)/urdf/VLP-16.urdf.xacro"/>
-  <VLP-16 parent="base_link" name="velodyne" topic="$(arg namespace)/velodyne_points" hz="10" samples="360" gpu="false" lasers="16" max_range="50">
-    <origin xyz="0 0 0.2" rpy="0 0 0" />
-  </VLP-16> -->
+  <VLP-16 parent="base_link" name="velodyne" topic="velodyne_points" hz="10" samples="1080" gpu="false" lasers="16" max_range="50">
+    <origin xyz="0 0 0.25" rpy="0 0 0" />
+  </VLP-16>
   <link name="land_pad">
     <visual>
