Commit message: Jackal with aruco marker on top

File: multi_jackal_description/urdf/custom_accessories.urdf.xacro (robot description, xacro)
@@ -5,4 +5,8 @@
        The accessory can then be enabled by setting the 'config' argument in the
        launch files. -->
+  <!-- Aruco markers. -->
+  <xacro:if value="$(optenv JACKAL_ARUCO 0)">
+    <xacro:include filename="accessories/aruco.urdf.xacro" />
+  </xacro:if>
   <!-- Box with AprilTag markers on each face. -->
   <xacro:if value="$(optenv JACKAL_APRILTAG 0)">

File: multi_jackal_description/urdf/jackal.urdf.xacro (robot description, xacro)
@@ -177,31 +177,63 @@
   <!-- Optional custom accessories. -->
   <xacro:include filename="custom_accessories.urdf.xacro" />
-  <!-- <xacro:include filename="$(find multi_jackal_description)/urdf/_d435.urdf.xacro" />
-  <sensor_d435 parent="base_link" name="rs_d435" topics_ns="$(arg namespace)/rs_d435" >
-    <origin xyz="0.4 0 0.2" rpy="0 0 0" />
-  </sensor_d435> -->
-  <xacro:include filename="$(find velodyne_description)/urdf/VLP-16.urdf.xacro"/>
-  <VLP-16 parent="base_link" name="velodyne" topic="velodyne_points" hz="10" samples="1080" gpu="false" lasers="16" max_range="50">
-    <origin xyz="0 0 0.25" rpy="0 0 0" />
-  </VLP-16>
+  <!-- Optional LANDING PAD -->
   <link name="land_pad">
-    <visual>
-      <geometry>
-        <box size="0.56 0.5 0.02"/>
+     <visual>
+       <geometry>
+         <box size="0.56 0.5 0.02"/>
+       </geometry>
+     </visual>
+     <collision>
+       <geometry>
+         <box size="0.56 0.5 0.02"/>
+       </geometry>
+     </collision>
+   </link>
+   <gazebo reference="land_pad">
+     <material>Gazebo/DarkGrey</material>
+   </gazebo>
+   <joint name="land_pad_link" type="fixed">
+     <parent link="base_link"/>
+     <child link="land_pad"/>
+     <origin xyz="0 0 0.2" rpy="0 0 0"/> <!-- original z=0.38 -->
+   </joint>
+  <!-- Optional ARUCO MARKER -->
+   <link name="tag_link">
+    <inertial>
+      <origin xyz="0 0 0" />
+      <mass value="0.001" />
+      <inertia  ixx="1.0" ixy="0.0"  ixz="0.0"  iyy="1.0"  iyz="0.0"  izz="1.0" />
+    </inertial>
+    <visual>
+      <origin xyz="0 0 0"/>
+      <geometry>
+        <mesh filename="package://multi_jackal_description/meshes/aruco/aruco_pattern.dae" scale="0.5 0.5 1" />
       </geometry>
     </visual>
     <collision>
-      <geometry>
-        <box size="0.56 0.5 0.02"/>
+      <origin xyz="0 0 0"/>
+      <geometry>
+        <box size="0.42 0.297 1e-05" /><!-- <box size="0.1778 0.1778 1e-05" />-->
       </geometry>
     </collision>
   </link>
-  <gazebo reference="land_pad">
-    <material>Gazebo/Black</material>
+  <joint name="aruco_joint" type="fixed">
+    <parent link="land_pad" />
+    <child link="tag_link" />
+    <origin xyz="0 0 0.02" rpy="0 0 0" /> <!-- z = land pad height -->
+    <axis xyz="0 1 0" />
+  </joint>
+  <xacro:property name="num" value="$(arg config_id)" />
+  <xacro:property name="width" value="0.005"/>
+  <link name="aruco_marker_0"></link>
+  <joint name="aruco_marker_0_joint" type="fixed">
+    <parent link="tag_link" />
+    <child link="aruco_marker_0" />
+    <origin xyz="0 0 ${width}" rpy="0 0 0"/>
+  </joint>
+<!--
+  <gazebo reference="base_link" >
+    <turnGravityOff>false</turnGravityOff>
   </gazebo>
-  <joint name="land_pad_link" type="fixed">
-    <parent link="base_link"/>
-    <child link="land_pad"/>
-    <origin xyz="0 0 0.38" rpy="0 0 0"/>
-  </joint>
+  -->
 </robot>
